File: design_files/AST1041.brd (EAGLE design)
At the start: 10 x 10 mm, 12 parts, among them J1 SM05B, U1 XC6210B18, U2 TX0102, U3 MAX30101

Commit message: updated documentation
Parts:
- C1: value 10uF -> 1uF; device tinycircuits:C0603 -> tinycircuits:C0402
- C3: value 10uF -> 0.1uF; device tinycircuits:C0603 -> tinycircuits:C0402
- C6: value 0.1uF -> 1uF
- J1: device tinycircuits:JST_SH_5X1 -> tinycircuits:JST_SH_5X1_EDGE
- U1: value XC6210B18 -> MAX30101; device tinycircuits:SOT-25@1 -> tinycircuits:MAX30100
- U3: value MAX30101 -> XC6210B18; device tinycircuits:MAX30100 -> tinycircuits:SOT-25
- moved C6 8.10 mm to (16.5, 22.9), turned to 180 degrees
- moved C4 4.95 mm to (21.2, 22.7), turned to 90 degrees
- moved C5 3.58 mm to (24.4, 21.1)
- moved U1 3.08 mm to (20.0, 19.0), flipped to the bottom, turned to 90 degrees
- moved U3 3.08 mm to (19.3, 22.0), flipped to the top, turned to 0 degrees
- moved C3 2.98 mm to (19.4, 22.6), flipped to the bottom, turned to 0 degrees
- moved C1 0.10 mm to (16.4, 20.0)
- moved C2 0.10 mm to (16.4, 21.1)
Connections:
- net 1V8: now also C6.1, U1.11, U3.5; no longer C5.1, U1.5, U3.11
- net GND: now also U1.12, U1.4, U3.2; no longer U1.2, U3.12, U3.4
- net N$1: now also U1.13; no longer U3.13
- net SCL_1V8: now also U1.2; no longer U3.2
- net SDA_1V8: now also U1.3; no longer U3.3
- net VCC: now also C5.1, U1.10, U1.9, U3.1, U3.3; no longer C6.1, U1.1, U1.3, U3.10, U3.9
Routing:
- net GND: track 2.86 -> 2.92 mm, vias 10 -> 11
Other:
- board text added: "Wireling Pulse Oximetry"
- board text removed: "Pulse Oximetry Sensor"
