File: design_files/AST1041.sch (EAGLE design)
At the start: 11 parts, among them J1 SM05B, U1 XC6210B18, U2 TX0102, U3 MAX30101

Commit message: updated documentation
Parts:
- C1: value 10uF -> 1uF; device tinycircuits:AS-ITM-00002 -> tinycircuits:AS-ITM-00105; PARTNO AS-ITM-00002 -> AS-ITM-00105; VALUE 10uF -> 1uF
- C3: value 10uF -> 0.1uF; device tinycircuits:AS-ITM-00002 -> tinycircuits:AS-ITM-00008; PARTNO AS-ITM-00002 -> AS-ITM-00008; VALUE 10uF -> 0.1uF
- C6: value 0.1uF -> 1uF; device tinycircuits:AS-ITM-00008 -> tinycircuits:AS-ITM-00105; PARTNO AS-ITM-00008 -> AS-ITM-00105; VALUE 0.1uF -> 1uF
- J1: device tinycircuits:AS-ITM-00340 -> tinycircuits:AS-ITM-00340EDGE
- U1: value XC6210B18 -> MAX30101; device tinycircuits:AS-ITM-00075 -> tinycircuits:AS-ITM-00473
- U3: value MAX30101 -> XC6210B18; device tinycircuits:AS-ITM-00473 -> tinycircuits:AS-ITM-00075
Connections:
- net 1V8: now also C6.1, U1.VDD, U3.VOUT; no longer C5.1, U1.VOUT, U3.VDD
- net GND: now also U1.GND, U1.PGND, U3.VSS; no longer U1.VSS, U3.GND, U3.PGND
- net N$1: now also U1.INT; no longer U3.INT
- net SCL_1V8: now also U1.SCL; no longer U3.SCL
- net SDA_1V8: now also U1.SDA; no longer U3.SDA
- net VCC: now also C5.1, U1.VLED+, U3.CE, U3.VIN; no longer C6.1, U1.CE, U1.VIN, U3.VLED+
Other:
- note added: "Variant: Standard - R"
- note added: "Wireling Pulse Oximetry"
- note removed: "Pulse Oximetry Sensor"
- note removed: "Variant: Standard"
- moved on the sheet: C3, C4, C5, C6
